File: Micromouse_PCB/Motor_Driver.kicad_sch (KiCad schematic)
At the start: 6 parts, among them U2 DRV8871DDA, U3 DRV8871DDA

Commit message: Schematic almost done, just need to do STM32 pinout
Changed lines of the file:
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@@
 	(wire
 		(pts
+			(xy 25.4 57.15) (xy 29.21 57.15)
+		)
+		(stroke
+			(width 0)
+			(type default)
+		)
+	)
+	(wire
+		(pts
 			(xy 121.92 33.02) (xy 128.27 33.02)
 		)
@@
 	(wire
 		(pts
+			(xy 25.4 25.4) (xy 29.21 25.4)
+		)
+		(stroke
+			(width 0)
+			(type default)
+		)
+	)
+	(wire
+		(pts
 			(xy 132.08 57.15) (xy 135.89 57.15)
 		)
@@
 	)
 	(label "Left_IN2"
-		(at 25.4 31.75 0)
+		(at 25.4 38.1 0)
 		(effects
 			(font
@@
 	)
 	(label "Left_IN1"
-		(at 25.4 25.4 0)
+		(at 25.4 31.75 0)
 		(effects
 			(font
@@
 	)
 	(label "Right_OUT2"
-		(at 177.8 44.45 180)
+		(at 177.8 50.8 180)
 		(effects
 			(font
@@
 	)
 	(label "Right_IN1"
-		(at 25.4 38.1 0)
+		(at 25.4 44.45 0)
 		(effects
 			(font
@@
 	)
 	(label "Left_OUT2"
-		(at 177.8 31.75 180)
+		(at 177.8 38.1 180)
 		(effects
 			(font
@@
 	)
 	(label "Right_OUT1"
-		(at 177.8 38.1 180)
+		(at 177.8 44.45 180)
 		(effects
 			(font
@@
 	)
 	(label "Right_IN2"
-		(at 25.4 44.45 0)
+		(at 25.4 50.8 0)
 		(effects
 			(font
@@
 	)
 	(label "Left_OUT1"
-		(at 177.8 25.4 180)
+		(at 177.8 31.75 180)
 		(effects
 			(font
@@
 	(hierarchical_label "Right_OUT2"
 		(shape output)
-		(at 177.8 44.45 0)
+		(at 177.8 50.8 0)
 		(effects
 			(font
@@
 		)
 	)
+	(hierarchical_label "GND"
+		(shape input)
+		(at 25.4 57.15 180)
+		(effects
+			(font
+				(size 1.27 1.27)
+			)
+			(justify right)
+		)
+	)
 	(hierarchical_label "Left_OUT1"
 		(shape output)
-		(at 177.8 25.4 0)
+		(at 177.8 31.75 0)
 		(effects
 			(font
@@
 	(hierarchical_label "Left_IN1"
 		(shape input)
-		(at 25.4 25.4 180)
+		(at 25.4 31.75 180)
 		(effects
 			(font
@@
 	(hierarchical_label "Right_IN2"
 		(shape input)
-		(at 25.4 44.45 180)
+		(at 25.4 50.8 180)
+		(effects
+			(font
+				(size 1.27 1.27)
+			)
+			(justify right)
+		)
+	)
+	(hierarchical_label "VBUS"
+		(shape input)
+		(at 25.4 25.4 180)
 		(effects
 			(font
@@
 	(hierarchical_label "Right_OUT1"
 		(shape output)
-		(at 177.8 38.1 0)
+		(at 177.8 44.45 0)
 		(effects
 			(font
@@
 	(hierarchical_label "Left_IN2"
 		(shape input)
-		(at 25.4 31.75 180)
+		(at 25.4 38.1 180)
 		(effects
 			(font
@@
 	(hierarchical_label "Right_IN1"
 		(shape input)
-		(at 25.4 38.1 180)
+		(at 25.4 44.45 180)
 		(effects
 			(font
@@
 	(hierarchical_label "Left_OUT2"
 		(shape output)
-		(at 177.8 31.75 0)
+		(at 177.8 38.1 0)
 		(effects
 			(font
@@
 	(symbol
 		(lib_id "power:GND")
+		(at 29.21 57.15 0)
+		(unit 1)
+		(exclude_from_sim no)
+		(in_bom yes)
+		(on_board yes)
+		(dnp no)
+		(fields_autoplaced yes)
+		(property "Reference" "#PWR057"
+			(at 29.21 63.5 0)
+			(effects
+				(font
+					(size 1.27 1.27)
+				)
+				(hide yes)
+			)
+		)
+		(property "Value" "GND"
+			(at 29.21 62.23 0)
+			(effects
+				(font
+					(size 1.27 1.27)
+				)
+			)
+		)
+		(property "Footprint" ""
+			(at 29.21 57.15 0)
+			(effects
+				(font
+					(size 1.27 1.27)
+				)
+				(hide yes)
+			)
+		)
+		(property "Datasheet" ""
+			(at 29.21 57.15 0)
+			(effects
+				(font
+					(size 1.27 1.27)
+				)
+				(hide yes)
+			)
+		)
+		(property "Description" "Power symbol creates a global label with name \"GND\" , ground"
+			(at 29.21 57.15 0)
+			(effects
+				(font
+					(size 1.27 1.27)
+				)
+				(hide yes)
+			)
+		)
+		(pin "1"
+		)
+		(instances
+			(project "Micromouse_PCB"
+				(path "/9f13efa1-6bd5-4a7e-a4ab-2916a4570f81/331c13d6-1eca-4c6d-9f54-5ae7f7b7b669"
+					(reference "#PWR057")
+					(unit 1)
+				)
+			)
+		)
+	)
+	(symbol
+		(lib_id "power:GND")
 		(at 91.44 62.23 0)
 		(unit 1)
@@
 					(unit 1)
 				)
+			)
+		)
+	)
+	(symbol
+		(lib_id "power:VBUS")
+		(at 29.21 25.4 0)
+		(unit 1)
+		(exclude_from_sim no)
+		(in_bom yes)
+		(on_board yes)
+		(dnp no)
+		(fields_autoplaced yes)
+		(property "Reference" "#PWR058"
+			(at 29.21 29.21 0)
+			(effects
+				(font
+					(size 1.27 1.27)
+				)
+				(hide yes)
+			)
+		)
+		(property "Value" "VBUS"
+			(at 29.21 20.32 0)
+			(effects
+				(font
+					(size 1.27 1.27)
+				)
+			)
+		)
+		(property "Footprint" ""
+			(at 29.21 25.4 0)
+			(effects
+				(font
+					(size 1.27 1.27)
+				)
+				(hide yes)
+			)
+		)
+		(property "Datasheet" ""
+			(at 29.21 25.4 0)
+			(effects
+				(font
+					(size 1.27 1.27)
+				)
+				(hide yes)
+			)
+		)
+		(property "Description" "Power symbol creates a global label with name \"VBUS\""
+			(at 29.21 25.4 0)
+			(effects
+				(font
+					(size 1.27 1.27)
+				)
+				(hide yes)
+			)
+		)
+		(pin "1"
+		)
+		(instances
+			(project "Micromouse_PCB"
+				(path "/9f13efa1-6bd5-4a7e-a4ab-2916a4570f81/331c13d6-1eca-4c6d-9f54-5ae7f7b7b669"
+					(reference "#PWR058")
+					(unit 1)
+				)

Commit message: Schematic done
Parts:
- R17, R18: footprint (none) -> Resistor_SMD:R_0603_1608Metric
Changed lines of the file:
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@@
 			)
 		)
-		(property "Footprint" ""
+		(property "Footprint" "Resistor_SMD:R_0603_1608Metric"
 			(at 91.44 59.69 0)
 			(effects
@@
 			)
 		)
-		(property "Footprint" ""
+		(property "Footprint" "Resistor_SMD:R_0603_1608Metric"
 			(at 135.89 59.69 0)
 			(effects
