File: Micromouse_PCB/Micromouse_PCB.kicad_pcb (KiCad board)
At the start: 2 copper layers, 104 parts, among them J1 Conn_01x06_MountingPin, J2 Conn_01x06_MountingPin, J3 ARM Cortex Debug, J4 Power, J5 ALARM PKLCS1212E, J6 USB-C, Q1 Q_NMOS_GSD, Q10 AA4040P3C-P22, Q11 Q_NMOS_GSD, Q12 Q_NMOS_GSD, Q13 AA4040P3C-P22, Q2 AA4040P3C-P22, Q3 Q_NMOS_GSD, Q4 AA4040P3C-P22, Q5 Q_NMOS_GSD, Q6 AA4040P3C-P22, Q7 Q_NMOS_GSD, Q8 AA4040P3C-P22, Q9 Q_NMOS_GSD, SW1 Slide switch, SW2 SW_Push, SW3 SW_Push, U1 STM32F105RCT6, U2 DRV8871DDA, U3 DRV8871DDA, U5 BMI088, U6 3V3_LDO AZ1117CH-3.3TRG1, U7 NCP1117-1.5_TO252, U8 USBLC6-2SC6, Y1 8MHz, OT32258MJBA4SL

Commit message: Placement 75% done on PCB
Parts:
- removed D14: SS34, Diode_SMD:D_SMA
- removed J6: USB-C, Connector_USB:USB_C_Receptacle_GCT_USB4105-xx-A_16P_TopMnt_Horizontal
- removed R22: 3.3k, Resistor_SMD:R_1206_3216Metric_Pad1.30x1.75mm_HandSolder
- removed R35, R38: 5.1K, Resistor_SMD:R_0603_1608Metric
- removed R39: 100k, Resistor_SMD:R_0603_1608Metric
- removed R40: 50k, Resistor_SMD:R_0603_1608Metric
- removed U8: USBLC6-2SC6, Package_TO_SOT_SMD:SOT-23-6
- added G***: LOGO, LOGO, F.Cu at (282.3, 58.7)
- added R19: 3.3k, Resistor_SMD:R_1206_3216Metric_Pad1.30x1.75mm_HandSolder, F.Cu at (190.5, 8.57)
- R15: value 35 -> 50Ω; footprint Resistor_SMD:R_1206_3216Metric_Pad1.30x1.75mm_HandSolder -> Resistor_SMD:R_0603_1608Metric
- SW1: footprint UCIRP-KiCAD-Lib:Horizontal_Slide_Swiitch SK12D07VG4NSPA_CNK -> Button_Switch_THT:SW_Slide-03_Wuerth-WS-SLTV_10x2.5x6.4_P2.54mm
- moved Q9 159.7 mm to (193.8, 7.91), turned to -90 degrees
- moved Q7 152.2 mm to (187.7, 7.91), turned to -90 degrees
- moved D5 150.8 mm to (193.9, 14.2)
- moved Q5 144.7 mm to (181.7, 7.91), turned to -90 degrees
- moved R14 143.3 mm to (193.2, 4.38), turned to 180 degrees
- moved D4 143.3 mm to (187.8, 14.2)
- moved R7 141.3 mm to (181.1, 4.38), turned to 180 degrees
- moved R15 140.3 mm to (192.5, 11.5), turned to 90 degrees
- moved D3 135.9 mm to (181.8, 14.2)
- moved R11 134.4 mm to (187.1, 4.38), turned to 180 degrees
- moved R13 131.9 mm to (184.5, 8.57), turned to 90 degrees
- moved R12 123.9 mm to (186.5, 11.5), turned to 90 degrees
- moved R10 122.9 mm to (178.4, 8.57), turned to 90 degrees
- moved Q8 118.4 mm to (183.1, 8.53)
- moved Q10 118.4 mm to (189.2, 8.53)
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Connections:
- net /PC0 renamed /STM32F105RCT6/PC0
- net /PC1 renamed /STM32F105RCT6/PC1
- net /PC10 renamed /STM32F105RCT6/PC10
- net /PC11 renamed /STM32F105RCT6/PC11
- net /PC12 renamed /STM32F105RCT6/PC12
- net /PC13 renamed /STM32F105RCT6/PC13
- net /PC14 renamed /STM32F105RCT6/PC14
- net /PC15 renamed /STM32F105RCT6/PC15
- net /PC2 renamed /STM32F105RCT6/PC2
- net /PC3 renamed /STM32F105RCT6/PC3
- net /PC4 renamed /STM32F105RCT6/PC4
- net /PC5 renamed /STM32F105RCT6/PC5
- net /PC6 renamed /STM32F105RCT6/PC6
- net /PC7 renamed /STM32F105RCT6/PC7
- net /PC8 renamed /STM32F105RCT6/PC8
- net /PC9 renamed /STM32F105RCT6/PC9
- J1 pad 2: /PB7 -> /STM32F105RCT6/PB7
- J1 pad 3: /PB6 -> /STM32F105RCT6/PB6
- J2 pad 2: /PB3 -> /STM32F105RCT6/PB3
- J2 pad 3: /PA15 -> /STM32F105RCT6/PA15
- Q1 pad 1: /PA4 -> /STM32F105RCT6/PA4
- Q12 pad 1: /PA3 -> /STM32F105RCT6/PA3
- Q13 pad 2: /PA2 -> /STM32F105RCT6/PA2
- Q2 pad 2: /PA1 -> /STM32F105RCT6/PA1
- Q3 pad 1: /PA5 -> /STM32F105RCT6/PA5
- Q4 pad 2: /PA0 -> /STM32F105RCT6/PA0
- Q5 pad 1: /PA6 -> /STM32F105RCT6/PA6
- Q7 pad 1: /PA7 -> /STM32F105RCT6/PA7
- R1 pad 1: /PA4 -> /STM32F105RCT6/PA4
- R11 pad 1: /PA7 -> /STM32F105RCT6/PA7
- R16 pad 1: /PA2 -> /STM32F105RCT6/PA2
- R20 pad 1: /PA3 -> /STM32F105RCT6/PA3
- R3 pad 1: /PA1 -> /STM32F105RCT6/PA1
- R36 pad 2: /PA10 -> /STM32F105RCT6/PA10
- R37 pad 1: /PA10 -> /STM32F105RCT6/PA10
- R4 pad 1: /PA5 -> /STM32F105RCT6/PA5
- R6 pad 1: /PA0 -> /STM32F105RCT6/PA0
- R7 pad 1: /PA6 -> /STM32F105RCT6/PA6
- U5 pad 1: /PB2 -> /STM32F105RCT6/PB2
- U5 pad 10: /PB14 -> /STM32F105RCT6/PB14
- U5 pad 12: /PB0 -> /STM32F105RCT6/PB0
- U5 pad 14: /PB12 -> /STM32F105RCT6/PB12
- U5 pad 15: /PB14 -> /STM32F105RCT6/PB14
- U5 pad 16: /PB10 -> /STM32F105RCT6/PB10
- U5 pad 5: /PB11 -> /STM32F105RCT6/PB11
- U5 pad 8: /PB13 -> /STM32F105RCT6/PB13
- U5 pad 9: /PB15 -> /STM32F105RCT6/PB15
Routing:
- net GND: track 0.00 -> 16.1 mm, vias 0 -> 12
- net /STM32F105RCT6/PA2: track 0.00 -> 3.94 mm
- net /STM32F105RCT6/PC3: track 0.00 -> 3.94 mm
- net /STM32F105RCT6/PC2: track 0.00 -> 3.94 mm
- net /STM32F105RCT6/PC1: track 0.00 -> 3.94 mm
- net /STM32F105RCT6/PA0: track 0.00 -> 3.94 mm
- net /STM32F105RCT6/PA1: track 0.00 -> 3.80 mm
- net /STM32F105RCT6/PA5: track 0.00 -> 2.60 mm
- net /STM32F105RCT6/PA3: track 0.00 -> 2.60 mm
- net /STM32F105RCT6/PC4: track 0.00 -> 2.60 mm
- net /STM32F105RCT6/PA7: track 0.00 -> 2.60 mm
- net /STM32F105RCT6/PA6: track 0.00 -> 2.60 mm
- net /STM32F105RCT6/PA4: track 0.00 -> 2.60 mm
- net Net-(Q12-D): track 0.00 -> 2.32 mm
- net Net-(Q9-D): track 0.00 -> 2.32 mm
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Other:
- board outline added: 120 x 93.4 mm
- board text added: "Battery"

Commit message: PCB Done, need review now
Parts:
- added G***: LOGO, LOGO, F.Cu at (89.0, 45.0)
- G***: moved to B.Cu
- J4: value Power -> Power XT30UPB-M; footprint Connector_AMASS:AMASS_XT30U-F_1x02_P5.0mm_Vertical -> Connector_AMASS:AMASS_XT30UPB-F_1x02_P5.0mm_Vertical
- moved G*** 191.2 mm to (91.2, 57.3), turned to 180 degrees
- moved SW2 175.9 mm to (62.1, 60.1)
- moved SW3 175.1 mm to (62.1, 67.6)
- moved R28 162.3 mm to (55.3, 60.1)
- moved R29 160.6 mm to (55.2, 67.6)
- moved D10 117.2 mm to (118.3, 65.0), turned to 180 degrees
- moved D9 115.0 mm to (118.3, 67.6), turned to 180 degrees
- moved D8 113.0 mm to (118.3, 70.2), turned to 180 degrees
- moved D6 111.3 mm to (118.3, 72.8), turned to 180 degrees
- moved R27 104.8 mm to (114.1, 67.6)
- moved R26 102.4 mm to (114.1, 70.2)
- moved R24 102.4 mm to (114.2, 65.0)
- moved R25 100.2 mm to (114.1, 72.8)
- moved R14 92.8 mm to (136.4, 77.8), turned to -90 degrees
- moved R7 88.1 mm to (107.4, 52.8)
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Connections:
- net 5V renamed +5V
- C1 pad 1: 3V3 -> +3V3
- C14 pad 1: 3V3 -> +3V3
- C15 pad 1: +3.3V -> +3V3
- C16 pad 1: +3.3V -> +3V3
- C18 pad 1: 3V3 -> +3V3
- C2 pad 1: 3V3 -> +3V3
- C3 pad 1: 3V3 -> +3V3
- C4 pad 1: 3V3 -> +3V3
- C5 pad 1: 3V3 -> +3V3
- C6 pad 1: 3V3 -> +3V3
- J3 pad 1: 3V3 -> +3V3
- J5 pad 1: +3.3V -> +3V3
- Q10 pad 1: 3V3 -> +3V3
- Q13 pad 1: 3V3 -> +3V3
- Q2 pad 1: 3V3 -> +3V3
- Q4 pad 1: 3V3 -> +3V3
- Q6 pad 1: 3V3 -> +3V3
- Q8 pad 1: 3V3 -> +3V3
- R28 pad 1: +3.3V -> +3V3
- R29 pad 1: +3.3V -> +3V3
- R32 pad 2: 3V3 -> +3V3
- R9 pad 2: 3V3 -> +3V3
- U1 pad 1: 3V3 -> +3V3
- U1 pad 13: 3V3 -> +3V3
- U1 pad 19: 3V3 -> +3V3
- U1 pad 32: 3V3 -> +3V3
- U1 pad 48: 3V3 -> +3V3
- U1 pad 64: 3V3 -> +3V3
- U6 pad 2: 3V3 -> +3V3
- Y1 pad 4: 3V3 -> +3V3
Routing:
- net +5V: track 0.00 -> 244.4 mm, vias 0 -> 9
- net VBUS: track 0.00 -> 145.1 mm, vias 0 -> 2
- net /STM32F105RCT6/PB7: track 0.00 -> 86.0 mm, vias 0 -> 2
- net /STM32F105RCT6/PB6: track 0.00 -> 83.6 mm, vias 0 -> 2
- net /STM32F105RCT6/PA2: track 3.94 -> 77.7 mm
- net GND: track 16.1 -> 87.9 mm, vias 12 -> 61
- net /STM32F105RCT6/PB14: track 0.00 -> 68.3 mm, vias 0 -> 3
- net /STM32F105RCT6/PB0: track 0.00 -> 63.7 mm, vias 0 -> 2
- net /STM32F105RCT6/PC5: track 0.00 -> 63.3 mm, vias 0 -> 2
- net /STM32F105RCT6/PB15: track 0.00 -> 62.3 mm, vias 0 -> 2
- net /STM32F105RCT6/PB13: track 0.00 -> 62.0 mm, vias 0 -> 2
- net /STM32F105RCT6/PA3: track 2.60 -> 62.8 mm
- net /STM32F105RCT6/PB2: track 0.00 -> 60.1 mm, vias 0 -> 2
- net /STM32F105RCT6/PC4: track 2.60 -> 62.1 mm, vias 0 -> 2
- net /STM32F105RCT6/PB10: track 0.00 -> 59.2 mm, vias 0 -> 2
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- added copper zone on F.Cu, net +3V3
- added copper zone on In2.Cu, net +3V3
- added copper zone on F.Cu, net +5V
- added copper zone on B.Cu, net GND
- added copper zone on F.Cu, net GND
- added copper zone on In1.Cu, net GND
Other:
- outline, holes or cut-outs redrawn
- copper layers 2 -> 4
- board text added: "Robert's Micromouse Spring 2026"
- board text added: "Set"
- board text added: "Start"
- board text added: "State1"
- board text added: "State2"
- board text added: "Thinking1"
- board text added: "Thinking2"

Commit message: Ordered
Parts:
- Q1, Q11, Q12, Q3, Q5, Q7, Q9: value Q_NMOS_GSD -> DMG3402LQ
- R12, R15, R2, R21, R5, R8: value 50Ω -> 50Ω 1.5W
- SW1: value Slide switch -> SW_SPDT; footprint Button_Switch_THT:SW_Slide-03_Wuerth-WS-SLTV_10x2.5x6.4_P2.54mm -> Button_Switch_THT:SW_Slide_SPDT_Straight_CK_OS102011MS2Q
- moved G*** 75.0 mm to (89.0, 120.0)
- moved G*** 17.5 mm to (90.9, 74.8)
- moved D5 10.0 mm to (136.6, 79.2)
- moved D7 10.0 mm to (41.4, 79.2)
- moved Q10 10.0 mm to (130.9, 74.5)
- moved Q12 10.0 mm to (47.7, 79.1)
- moved Q13 10.0 mm to (47.0, 74.5)
- moved Q9 10.0 mm to (130.3, 77.2)
- moved R14 10.0 mm to (126.4, 77.8)
- moved R15 10.0 mm to (133.8, 80.6)
- moved R16 10.0 mm to (47.0, 75.9)
- moved R19 10.0 mm to (130.8, 73.2)
- moved R20 10.0 mm to (51.2, 78.5)
- moved R21 10.0 mm to (44.1, 77.9)
- moved D2 9.25 mm to (68.0, 52.5)
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Connections:
- C11 pad 1: 3V3 -> +3V3
- C13 pad 1: 3V3 -> +3V3
- SW1 pad 1: Net-(J4-Pin_2) -> Net-(SW1-A)
- SW1 pad 2: GND -> Net-(J4-Pin_2)
- SW1 pad 3: Net-(SW1-A) -> GND
- U5 pad 11: 3V3 -> +3V3
- U5 pad 3: 3V3 -> +3V3
Routing:
- net +5V: track 244.4 -> 205.9 mm
- net /STM32F105RCT6/PC4: track 62.1 -> 51.8 mm
- net +3V3: track 47.5 -> 56.9 mm, vias 36 -> 38
- net 3V3: track 9.35 -> 0.00 mm
- net /STM32F105RCT6/PA3: track 62.8 -> 54.6 mm
- net /STM32F105RCT6/PA7: track 52.7 -> 45.6 mm
- net /STM32F105RCT6/PA2: track 77.7 -> 72.3 mm
- net /STM32F105RCT6/PA4: track 51.2 -> 46.0 mm
- net /STM32F105RCT6/PC3: track 23.5 -> 19.2 mm
- net /STM32F105RCT6/PA1: track 61.8 -> 57.8 mm
- net /STM32F105RCT6/PC11: track 27.9 -> 24.2 mm
- net /STM32F105RCT6/PC10: track 27.3 -> 24.1 mm
- net GND: track 87.9 -> 90.6 mm
- net /STM32F105RCT6/PC12: track 28.6 -> 26.7 mm
- net /STM32F105RCT6/PC13: track 19.9 -> 18.1 mm
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Other:
- board size 120 x 93.4 mm -> 100 x 84.9 mm
- board text added: "1"
- board text added: "3V3"
- board text added: "5V"
- board text added: "BUZZER"
- board text added: "OFF"
- board text added: "ON"
- board text added: "VBUS"
- board text removed: "Battery"
