File: Micromouse_PCB/One_Emitter_Receiver.kicad_sch (KiCad schematic)
At the start: 6 parts, among them Q1 Q_NMOS_GSD, Q2 AA4040P3C-P22

Commit message: PCB Done, need review now
Parts:
- R2: value 50Ω -> 50Ω 1W
Other:
- moved on the sheet: D1, Q1, Q2, R1, R2, R3

Commit message: Ordered
Parts:
- Q1: value Q_NMOS_GSD -> DMG3402LQ
- R2: value 50Ω 1W -> 50Ω 1.5W
Changed lines of the file:
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@@
 			)
 		)
-		(property "Value" "Q_NMOS_GSD"
+		(property "Value" "DMG3402LQ"
 			(at 85.1916 43.053 0)
 			(effects
@@
 			)
 		)
-		(property "Value" "50Ω 1W"
+		(property "Value" "50Ω 1.5W"
 			(at 85.344 34.0614 0)
 			(effects
