File: Micromouse_PCB/PDN.kicad_sch (KiCad schematic)
At the start: 12 parts, among them U6 3V3_LDO AZ1117CH-3.3TRG1, U7 NCP1117-1.5_TO252

Commit message: PCB Done, need review now
Connections:
- net 3V3 renamed +3V3
- net 5V renamed +5V
Changed lines of the file:
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@@
 			)
 		)
-		(property "Value" "5V"
+		(property "Value" "+5V"
 			(at 171.45 21.59 0)
 			(effects
@@
 			)
 		)
-		(property "Value" "5V"
+		(property "Value" "+5V"
 			(at 77.47 63.5 0)
 			(effects
@@
 			)
 		)
-		(property "Value" "5V"
+		(property "Value" "+5V"
 			(at 127 22.86 0)
 			(effects
@@
 			)
 		)
-		(property "Value" "3V3"
+		(property "Value" "+3V3"
 			(at 171.45 34.29 0)
 			(effects
@@
 			)
 		)
-		(property "Value" "3V3"
+		(property "Value" "+3V3"
 			(at 127 63.5 0)
 			(effects
